Commit message: urdf on camera and objects

File: urdf/objects/bar_clamp.urdf.xacro (robot description, xacro)
@@ -3,12 +3,12 @@
   <link name="bar_clamp">
     <visual>
-       <geometry>
-	  <mesh filename="package://gqcnn_demo/meshes/objects/bar_clamp.dae"/>
-	</geometry>
+      <geometry>
+	      <mesh filename="package://gqcnn_demo/meshes/objects/bar_clamp.dae"/>
+	    </geometry>
     </visual>
     <collision>
-       <geometry>
-       <mesh filename="package://gqcnn_demo/meshes/objects/bar_clamp.dae"/>
-	</geometry>
+      <geometry>
+        <mesh filename="package://gqcnn_demo/meshes/objects/bar_clamp.dae"/>
+	    </geometry>
     </collision>
 	<inertial>
@@ -21,6 +21,6 @@
       <kp>1000000</kp>
       <kd>1.0</kd>
-      <mu1>100.0</mu1>
-      <mu2>100.0</mu2>
+      <mu1>1000.0</mu1>
+      <mu2>1000.0</mu2>
       <minDepth>0.001</minDepth>
   </gazebo>

File: urdf/panda_camera.urdf.xacro (robot description, xacro)
@@ -29,16 +29,16 @@
   <xacro:property name="cam_oy" value="0.0" />
   <link name="camera_link">
-      <visual>
+      <!-- <visual>
        <origin xyz="0 0 0" rpy="0 0 ${M_PI/2}"/>
         <geometry>
-         <mesh filename="package://gqcnn_demo/meshes/kinect.dae"/>
+         <mesh filename="package://gqcnn_demo/meshes/camera/kinect.dae"/>
         </geometry>
       </visual>
       <collision>
-        <origin xyz="0.0 0.0 0.0" rpy="0 0 0"/>
+        <origin xyz="0 0 0" rpy="0 0 ${M_PI/2}"/>
         <geometry>
-          <box size="0.07271 0.27794 0.073"/>
+          <mesh filename="package://gqcnn_demo/meshes/camera/kinect.dae"/>
         </geometry>
-      </collision>
+      </collision> -->
       <inertial>
         <mass value="0.564" />
