Commit message: update mesh file

File: deep_grasp_task/urdf/objects/bar_clamp.urdf.xacro (robot description, xacro)
@@ -4,10 +4,10 @@
     <visual>
       <geometry>
-	      <mesh filename="package://gqcnn_demo/meshes/objects/bar_clamp.dae"/>
+	      <mesh filename="package://deep_grasp_task/meshes/objects/bar_clamp.dae"/>
 	    </geometry>
     </visual>
     <collision>
       <geometry>
-        <mesh filename="package://gqcnn_demo/meshes/objects/bar_clamp.dae"/>
+        <mesh filename="package://deep_grasp_task/meshes/objects/bar_clamp.dae"/>
 	    </geometry>
     </collision>

File: deep_grasp_task/urdf/objects/strawberry.urdf.xacro (robot description, xacro)
@@ -4,10 +4,10 @@
   <visual>
      <geometry>
-	       <mesh filename="package://gqcnn_demo/meshes/objects/strawberry.dae"/>
+	       <mesh filename="package://deep_grasp_task/meshes/objects/strawberry.dae"/>
 	     </geometry>
   </visual>
   <collision>
     <geometry>
-       <mesh filename="package://gqcnn_demo/meshes/objects/strawberry.dae"/>
+       <mesh filename="package://deep_grasp_task/meshes/objects/strawberry.dae"/>
 	   </geometry>
   </collision>
