Commit message: remove material tag

File: deep_grasp_task/urdf/objects/cylinder.urdf.xacro (robot description, xacro)
@@ -25,5 +25,5 @@
   </link>
   <gazebo reference="cylinder_link">
-    <material>Gazebo/Green</material>
+    <!-- <material>Gazebo/Grey</material> -->
     <dampingFactor>0.005</dampingFactor>
     <kp>1000000</kp>
