Commit message: removed comment block:

File: deep_grasp_task/urdf/robots/panda_camera.urdf.xacro (robot description, xacro)
@@ -17,10 +17,3 @@
     <mu2>100.0</mu2>
   </gazebo>
-  <!-- overhead position -->
-  <!-- <xacro:property name="cam_px" value="0.5" />
-  <xacro:property name="cam_py" value="0.0" />
-  <xacro:property name="cam_pz" value="0.7" />
-  <xacro:property name="cam_or" value="0.0" />
-  <xacro:property name="cam_op" value="${M_PI/2.0}" />
-  <xacro:property name="cam_oy" value="0.0" /> -->
 </robot>
